File: circuit/berlingo synth 0.5.sch (EAGLE design)
At the start: 61 parts, among them SW1 OS102011MA1Q

Commit message: Berlingo Synth 0.5 and 0.6
Parts:
- removed INL_C1, INR_C1, LFO_C1: 226, SparkFun-Capacitors:CAPEZ
- removed LED_C1: 100uF, rcl:CPOL-USE2-4
- removed LED_C2: 100uF, rcl:CPOL-USE2.5-6
- added 9V+: KEYSTONE-629+, kanflo:KEYSTONE-629+
- added FILTER_IN1, FILTER_OUT1, INL1, INR1, LFO1, LFO_A, LFO_B, LFO~, OUTL1, OUTR1, PWM_A, PWM_B, PWM_IN1, PWM_OUT1, VCO1, VCO_A, VCO_B, VCO~1, ~LED1, ~PWM1: (no value), TOF:HEADER-1X1
- added GND: KEYSTONE-629, kanflo:KEYSTONE-629
- added INL_C, INR_C: 10-22uF, adafruit:C-US025-024X044
- added LFO_C: 22uF, rcl:CPOL-USE2.5-6
- added LFO~1: ~LFO, TOF:HEADER-1X1
- OUTL_C1, OUTR_C1: value 226 -> 10-22uF; device SparkFun-Capacitors:CAPEZ -> adafruit:C-US025-024X044
Connections:
- net FILTER_IN: now also FILTER_IN1.1
- net FILTER_OUT: now also FILTER_OUT1.1
- net GND: now also GND.GND, LFO_C.-; no longer LED_C1.-, LFO_C1.2
- net LFO: now also LFO1.1
- net MOD_IN: now also PWM_IN1.1
- net N$1: now also 9V+.V+
- net N$10: now also VCO_B.1
- net N$12: now also OUTL1.1
- net N$13: now also ~LED1.1; no longer LED_C1.+
- net N$14: now also INR1.1, INR_C.1; no longer INR_C1.1
- net N$15: now also INR_C.2; no longer INR_C1.2
- net N$18: now also VCO_A.1
- net N$19: now also INL1.1, INL_C.1; no longer INL_C1.1
- net N$20: now also INL_C.2; no longer INL_C1.2
- net N$21: now also LFO_B.1
- net N$22: now also LFO_A.1, LFO_C.+, LFO~.1, LFO~1.1; no longer LFO_C1.1
- net N$23: now also VCO1.1
- net N$3: now also PWM_A.1
- net N$5: now also ~PWM1.1
- net N$9: now also OUTR1.1
- net PWM_OUT: now also PWM_B.1, PWM_OUT1.1
- net TRIANGLE_PITCHMOD: now also VCO~1.1
Other:
- moved on the sheet: H3
