File: circuit/op-synth 0.8.sch (EAGLE design)
At the start: 77 parts, among them SW1 OS102011MA1QOS102011MA1Q_TOP

Commit message: Version 0.8
Parts:
- INL_C, INR_C, LFO_C, OUTL_C1, OUTR_C1: value 22uF -> 226
Changed lines of the file:
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@@
 <part name="SUPPLY3" library="SparkFun-Aesthetics" deviceset="VIN" device=""/>
 <part name="GND8" library="SparkFun-Aesthetics" deviceset="GND" device=""/>
-<part name="LFO_C" library="resistor" deviceset="C-US" device="050-024X044" value="22uF"/>
-<part name="INL_C" library="adafruit" deviceset="C-US" device="050-024X044" value="22uF"/>
-<part name="INR_C" library="adafruit" deviceset="C-US" device="050-024X044" value="22uF"/>
-<part name="OUTL_C1" library="adafruit" deviceset="C-US" device="050-024X044" value="22uF"/>
-<part name="OUTR_C1" library="adafruit" deviceset="C-US" device="050-024X044" value="22uF"/>
+<part name="LFO_C" library="resistor" deviceset="C-US" device="050-024X044" value="226"/>
+<part name="INL_C" library="adafruit" deviceset="C-US" device="050-024X044" value="226"/>
+<part name="INR_C" library="adafruit" deviceset="C-US" device="050-024X044" value="226"/>
+<part name="OUTL_C1" library="adafruit" deviceset="C-US" device="050-024X044" value="226"/>
+<part name="OUTR_C1" library="adafruit" deviceset="C-US" device="050-024X044" value="226"/>
 <part name="VCO~1" library="TOF" deviceset="HEADER-1X1" device=""/>
 <part name="VCO1" library="TOF" deviceset="HEADER-1X1" device=""/>
