File: circuit/op-synth 2018-05-09.sch (EAGLE design)
At the start: 78 parts, among them SW1 OS102011MA1QOS102011MA1Q_TOP

Commit message: New version
Parts:
- removed INL_R1, INL_R2: 100k, resistor:R-US_0204/7
- removed INR_R1, INR_R2: 10k, resistor:R-US_0204/7
- added PWM_R3, PWM_R4: 10k, resistor:R-US_0204/7
- LED_R1: value 150 -> 330
- PWM_IN, PWM_OUT: value PWM -> AMP
- VCO: value VCO -> OSC
- VCO~: value VCO~ -> OSC~
- ~PWM: value PWM~ -> AMP~
Connections:
- removed net N$25 (its old number): ATTENUATION.S, FX_ICA.-IN, INR_R1.2
- removed net N$26: FX_ICA.OUT, INR_R2.1, PWM_OUT.1, PWM_OUT1.1
- new net N$5: ATTENUATION.A, PWM_R4.1
- new net PWM_OUT: FX_ICA.OUT, PWM_OUT.1, PWM_OUT1.1, PWM_R4.2
- net MOD_IN: now also PWM_R3.1; no longer INR_R1.1
- net N$3: now also ATTENUATION.S, FX_ICA.-IN, PWM_R3.2; no longer ATTENUATION.A, INR_R2.2
Other:
- note added: "Warning: Use eagle 6.6 to export"
- note removed: "Use eagle 6.6 to export"
- moved on the sheet: ATTENUATION, FI_C1, PWM_IN, PWM_IN1, PWM_OUT, PWM_OUT1, PWM_R1, PWM_R2, P_LED, ~PWM, ~PWM1
