File: circuit/op-synth.sch (EAGLE design)
At the start: 76 parts, among them SW1 OS102011MA1QOS102011MA1Q_TOP

Commit message: Updated to latest version
Parts:
- removed 9V+: KEYSTONE-629+, kanflo:KEYSTONE-629+
- removed GND: KEYSTONE-629, kanflo:KEYSTONE-629
- removed PWM_R3, PWM_R4: 10k, resistor:R-US_0204/7
- added 9V_+: KEYSTONE-637, kanflo:KEYSTONE-637
- added 9V_GND: KEYSTONE-629, kanflo:KEYSTONE-629
- added INL_R1, INL_R2: 100k, resistor:R-US_0204/7
- added INR_R1, INR_R2: 10k, resistor:R-US_0204/7
- LED_R1: value 330 -> 150
- PWM_IN, PWM_OUT: value AMP -> PWM
- VCO: value OSC -> VCO
- VCO~: value OSC~ -> VCO~
- ~PWM: value AMP~ -> PWM~
Connections:
- removed net MOD_IN: PWM_IN.1, PWM_IN1.1, PWM_R3.1
- removed net N$5 (its old number): ATTENUATION.A, PWM_R4.1
- removed net PWM_OUT: FX_ICA.OUT, PWM_OUT.1, PWM_OUT1.1, PWM_R4.2
- new net N$25: ATTENUATION.S, FX_ICA.-IN, INL_R1.2
- new net N$26: FX_ICA.OUT, INL_R2.1, PWM_OUT.1, PWM_OUT1.1
- new net N$27: INR_R2.2, OUTR_C1.1
- new net N$28: INR_R1.2, OUTL.1, OUTL1.1
- new net N$30: INR_R1.1, OUTL_C1.1
- net GND: now also 9V_GND.GND; no longer GND.GND
- net N$1: now also 9V_+.VCC; no longer 9V+.V+
- net N$12: now also INL_R1.1, PWM_IN.1, PWM_IN1.1; no longer OUTL.1, OUTL1.1, OUTL_C1.1
- net N$3: now also ATTENUATION.A, INL_R2.2; no longer ATTENUATION.S, FX_ICA.-IN, PWM_R3.2
- net N$9: now also INR_R2.1; no longer OUTR_C1.1
Other:
- note added: "Use eagle 6.6 to export"
- note removed: "Warning: Use eagle 6.6 to export"
- moved on the sheet: ATTENUATION, FI_C1, OUTL, OUTL1, OUTR, OUTR1, PWM_IN, PWM_IN1, PWM_OUT, PWM_OUT1, PWM_R1, PWM_R2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
